File: KiCad/sensors/RP-008295-DS-1-Minimal-KiCAD rp2350/RP-006440-DD-2-RP2350A Minimal Board Kicad archive/_autosave-RP2350_electrophy2.kicad_sch (KiCad schematic)
At the start: 100 parts, among them J1 INA INPUT, J10 BATTERY, J11 Conn_01x06_Pin, J12 Conn_01x02_Pin, J2 Conn_02x18_Odd_Even, J3 Conn_02x18_Odd_Even, J4 SM03B-SRSS-TB, J5 USB_C_Receptacle_USB2.0_16P, J6 BATTERY, J7 Conn_01x02_Pin, J8 Conn_01x04_Pin, J9 Conn_01x06_Pin, SW1 SW_Push, SW2 SW_Push, SW3 SW_Push, U1 RP2350_60QFN, U2 MCP1700x-330xxTO, U3 W25Q128JVS, U4 VL53L0CXV0DH1, U5 INA219AxD, U6 USBLC6-2P6, U7 ESP-12F, U8 W25Q128JVS, U9 AMS1117-3.3, Y2 Crystal

Commit message: a
Parts:
- added SW4: SW_Push, Button_Switch_SMD:SW_SPST_TL3305A, symbol Switch:SW_Push
Connections:
- net +3.3V: now also SW4.1
- net GND: now also SW4.2
Other:
- note added: "boot"
- note added: "flash"
- note added: "reset"
Changed lines of the file:
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@@
 		)
 	)
+	(text "boot\n"
+		(exclude_from_sim no)
+		(at 119.634 132.08 0)
+		(effects
+			(font
+				(size 1.27 1.27)
+			)
+		)
+	)
 	(text "LIPO BATTERY\n"
 		(exclude_from_sim no)
@@
 		)
 	)
+	(text "reset\n"
+		(exclude_from_sim no)
+		(at 59.69 77.724 0)
+		(effects
+			(font
+				(size 1.27 1.27)
+			)
+		)
+	)
 	(text "POWER MANAGEMENT\n"
 		(exclude_from_sim no)
@@
 		)
 	)
+	(text "flash\n"
+		(exclude_from_sim no)
+		(at 135.128 30.988 0)
+		(effects
+			(font
+				(size 1.27 1.27)
+			)
+		)
+	)
 	(text "POWER MANAGEMENT\n"
 		(exclude_from_sim no)
@@
 	)
 	(junction
+		(at 129.54 36.83)
+		(diameter 0)
+		(color 0 0 0 0)
+	)
+	(junction
 		(at 107.95 90.17)
 		(diameter 0)
@@
 	(wire
 		(pts
+			(xy 133.35 36.83) (xy 129.54 36.83)
+		)
+		(stroke
+			(width 0)
+			(type default)
+		)
+	)
+	(wire
+		(pts
 			(xy 234.95 60.96) (xy 246.38 60.96)
 		)
@@
 	(wire
 		(pts
+			(xy 129.54 35.56) (xy 129.54 36.83)
+		)
+		(stroke
+			(width 0)
+			(type default)
+		)
+	)
+	(wire
+		(pts
 			(xy 339.09 226.06) (xy 326.39 226.06)
 		)
@@
 	(wire
 		(pts
+			(xy 129.54 36.83) (xy 119.38 36.83)
+		)
+		(stroke
+			(width 0)
+			(type default)
+		)
+	)
+	(wire
+		(pts
 			(xy 229.87 104.14) (xy 241.3 104.14)
 		)
@@
 		)
 		(property "Value" "5K"
-			(at 116.078 30.226 0)
+			(at 116.078 32.258 0)
 			(effects
 				(font
@@
 				)
 				(justify left)
-				(hide yes)
 			)
 		)
@@
 	)
 	(symbol
+		(lib_id "Switch:SW_Push")
+		(at 129.54 30.48 90)
+		(unit 1)
+		(exclude_from_sim no)
+		(in_bom yes)
+		(on_board yes)
+		(dnp no)
+		(property "Reference" "SW4"
+			(at 120.396 29.972 90)
+			(effects
+				(font
+					(size 1.27 1.27)
+				)
+				(justify right)
+			)
+		)
+		(property "Value" "SW_Push"
+			(at 119.38 32.766 90)
+			(effects
+				(font
+					(size 1.27 1.27)
+				)
+				(justify right)
+			)
+		)
+		(property "Footprint" "Button_Switch_SMD:SW_SPST_TL3305A"
+			(at 124.46 30.48 0)
+			(effects
+				(font
+					(size 1.27 1.27)
+				)
+				(hide yes)
+			)
+		)
+		(property "Datasheet" "~"
+			(at 124.46 30.48 0)
+			(effects
+				(font
+					(size 1.27 1.27)
+				)
+				(hide yes)
+			)
+		)
+		(property "Description" "Push button switch, generic, two pins"
+			(at 129.54 30.48 0)
+			(effects
+				(font
+					(size 1.27 1.27)
+				)
+				(hide yes)
+			)
+		)
+		(pin "1"
+		)
+		(pin "2"
+		)
+		(instances
+			(project "RP2350_electrophy2"
+				(path "/94683f5c-9cd9-448e-be96-9792537b5cb8"
+					(reference "SW4")
+					(unit 1)
+				)
+			)
+		)
+	)
+	(symbol
 		(lib_id "Device:C")
 		(at 292.1 66.04 0)
@@
 	(symbol
 		(lib_id "power:+3.3V")
-		(at 119.38 36.83 270)
+		(at 133.35 36.83 270)
 		(unit 1)
 		(exclude_from_sim no)
@@
 		(fields_autoplaced yes)
 		(property "Reference" "#PWR060"
-			(at 115.57 36.83 0)
+			(at 129.54 36.83 0)
 			(effects
 				(font
@@
 		)
 		(property "Value" "+3.3V"
-			(at 123.19 36.8299 90)
+			(at 137.16 36.8299 90)
 			(effects
 				(font
@@
 		)
 		(property "Footprint" ""
-			(at 119.38 36.83 0)
+			(at 133.35 36.83 0)
 			(effects
 				(font
@@
 		)
 		(property "Datasheet" ""
-			(at 119.38 36.83 0)
+			(at 133.35 36.83 0)
 			(effects
 				(font
@@
 		)
 		(property "Description" "Power symbol creates a global label with name \"+3.3V\""
-			(at 119.38 36.83 0)
+			(at 133.35 36.83 0)
 			(effects
 				(font
@@
 		)
 		(property "Value" "5K"
-			(at 124.968 42.926 0)
+			(at 126.238 44.704 0)
 			(effects
 				(font
@@
 					(unit 1)
 				)
+			)
+		)
+	)
+	(symbol
+		(lib_id "power:GND")
+		(at 129.54 25.4 180)
+		(unit 1)
+		(exclude_from_sim no)
+		(in_bom yes)
+		(on_board yes)
+		(dnp no)
+		(fields_autoplaced yes)
+		(property "Reference" "#PWR074"
+			(at 129.54 19.05 0)
+			(effects
+				(font
+					(size 1.27 1.27)
+				)
+				(hide yes)
+			)
+		)
+		(property "Value" "GND"
+			(at 129.54 20.32 0)
+			(effects
+				(font
+					(size 1.27 1.27)
+				)
+			)
+		)
+		(property "Footprint" ""
+			(at 129.54 25.4 0)
+			(effects
+				(font
+					(size 1.27 1.27)
+				)
+				(hide yes)
+			)
+		)
+		(property "Datasheet" ""
+			(at 129.54 25.4 0)
+			(effects
+				(font
+					(size 1.27 1.27)
+				)
+				(hide yes)
+			)
+		)
+		(property "Description" "Power symbol creates a global label with name \"GND\" , ground"
+			(at 129.54 25.4 0)
+			(effects
+				(font
+					(size 1.27 1.27)
+				)
+				(hide yes)
+			)
+		)
+		(pin "1"
+		)
+		(instances
+			(project "RP2350_electrophy2"
+				(path "/94683f5c-9cd9-448e-be96-9792537b5cb8"
+					(reference "#PWR074")
+					(unit 1)
+				)
